File: Seadream Avionics Barney/Seadream Avionics Barney.kicad_pcb (KiCad board)
At the start: 2 copper layers, 26 x 63 mm, 41 parts, among them J1 B2B-PH-K-S(LF)(SN), J2 C393939, J3 B2B-PH-K-S(LF)(SN), SW1 SSSS810701, U1 BMP280, U2 ESP32-S3-MINI-1U-N8, U3 LSM6DSO32TR, U4 LD1117S33TR, U5 SHT40-AD1B-R3, U6 LD39200PU33R, U7 MAX98357AETE_T

Commit message: Added logo
Parts:
- added G***: LOGO, Downloads:twst, B.Cu at (157.5, 80.2)
